File: kicad/ledStripDriver.sch (KiCad schematic (older format))
At the start: 57 parts, among them J1 AudioJack3_SwitchTR, J2 USB_POWER_OUT, K1 G5RL1AELN5DC, Q1 Q_NPN_BEC_S8050, Q2 AO3400, Q3 AO3400, Q4 AO3400, SW1 SW_DIP_x01, SW2 Rotary_Encoder_Switch, SW3 SW_Push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

Commit message: Rainbow is pulsing. MDNS correctly configured. drawMap(...) is not injecting any delay.
Parts:
- removed Q1: Q_NPN_BEC_S8050, Package_TO_SOT_SMD:SOT-23, symbol Device:Q_NPN_BEC
- removed R1: ~47ohm, Resistor_SMD:R_0805_2012Metric_Pad1.15x1.40mm_HandSolder, symbol Device:R
- removed R_ENC_A1, R_ENC_B1: 10k, Resistor_SMD:R_0805_2012Metric_Pad1.15x1.40mm_HandSolder, symbol Device:R
- added D4: D_Schottky, Diode_SMD:D_SMA_Handsoldering, symbol Device:D_Schottky
- added Q1: AO3400A, Package_TO_SOT_SMD:SOT-23, symbol Transistor_FET:AO3400A
- R_LS1_12V1, R_LS2_12V1, R_LS3_12V1: value 4k7 -> 1k
Connections:
- wire segments 197 -> 195
- no-connect marks 23 -> 22
Other:
- moved on the sheet: C_GND_MSGEQ7, R_EQ_V_DIV1, R_EQ_V_DIV2
