File: kicad/ledStripDriver.kicad_pcb (KiCad board)
At the start: 2 copper layers, 110 x 91 mm, 57 parts, among them J1 AudioJack3_SwitchTR, J2 USB_POWER_OUT, K1 G5RL1AELN5DC, Q1 Q_NPN_BEC_S8050, Q2 AO3400, Q3 AO3400, Q4 AO3400, SW1 SW_DIP_x01, SW2 Rotary_Encoder_Switch, SW3 SW_Push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

Commit message: Rainbow is pulsing. MDNS correctly configured. drawMap(...) is not injecting any delay.
Parts:
- removed R1: ~47ohm, Resistor_SMD:R_0805_2012Metric_Pad1.15x1.40mm_HandSolder
- removed R_ENC_A1, R_ENC_B1: 10k, Resistor_SMD:R_0805_2012Metric_Pad1.15x1.40mm_HandSolder
- added D4: D_Schottky, Diode_SMD:D_SMA_Handsoldering, F.Cu at (122.9, 80.5)
- Q1: value Q_NPN_BEC_S8050 -> AO3400A
- R_L2_12V1: renamed from R9; value R_L2_12V -> 300
- R_LS1_12V1, R_LS2_12V1, R_LS3_12V1: value 4k7 -> 1k
- moved Q1 11.6 mm to (110.2, 74.1), turned to 90 degrees
- moved D3 8.04 mm to (116.5, 71.6)
- moved K1 5.31 mm to (134.3, 70.3)
- moved R_EQ_V_DIV1 3.99 mm to (158.7, 133.8), turned to 90 degrees
- moved R_EQ_V_DIV2 2.03 mm to (159.0, 137.6)
Connections:
- D3 pad 2: GND -> Net-(D3-Pad2)
- K1 pad 8: GND -> Net-(D3-Pad2)
- Q1 pad 1: Net-(Q1-Pad1) -> /RELAY_DRIVER
- Q1 pad 2: Net-(D3-Pad1) -> GND
- Q1 pad 3: +5V -> Net-(D3-Pad2)
- R_EQ_V_DIV1 pad 1: GND -> Net-(R_EQ_V_DIV1-Pad1)
- R_EQ_V_DIV1 pad 2: Net-(R_EQ_V_DIV1-Pad2) -> GND
- R_EQ_V_DIV2 pad 1: Net-(R_EQ_V_DIV1-Pad2) -> Net-(R_EQ_V_DIV2-Pad1)
- R_EQ_V_DIV2 pad 2: Net-(R_EQ_V_DIV2-Pad2) -> Net-(R_EQ_V_DIV1-Pad1)
- U1 pad 10: Net-(R_ENC_B1-Pad1) -> Net-(C_ENC_B1-Pad1)
- U1 pad 11: Net-(R_ENC_A1-Pad1) -> Net-(C_ENC_A1-Pad1)
- U1 pad 14: Net-(U1-Pad14) -> GND
- U1 pad 20: Net-(U1-Pad14) -> GND
- U1 pad 26: Net-(U1-Pad14) -> GND
- U1 pad 27: (no net) -> /RELAY_DRIVER
- U1 pad 32: Net-(R_EQ_V_DIV1-Pad2) -> (no net)
- U1 pad 35: /RELAY_DRIVER -> (no net)
- U1 pad 5: (no net) -> Net-(R_EQ_V_DIV2-Pad1)
- U3 pad 3: Net-(R_EQ_V_DIV2-Pad2) -> Net-(R_EQ_V_DIV1-Pad1)
Routing:
- net Net-(C_ENC_B1-Pad1): track 13.0 -> 102.1 mm
- net Net-(R_ENC_B1-Pad1): track 88.8 -> 0.00 mm
- net Net-(R_ENC_A1-Pad1): track 88.5 -> 0.00 mm
- net Net-(C_ENC_A1-Pad1): track 19.7 -> 106.7 mm, vias 2 -> 3
- net GND: track 94.1 -> 153.3 mm
- net Net-(R_EQ_V_DIV2-Pad1): track 0.00 -> 52.7 mm, vias 0 -> 2
- net /12V_PRE_RELAY: track 47.3 -> 97.9 mm
- net Net-(U1-Pad14): track 48.9 -> 0.00 mm
- net Net-(R_EQ_V_DIV1-Pad2): track 46.1 -> 0.00 mm
- net /RELAY_DRIVER: track 54.3 -> 74.0 mm
- net Net-(D3-Pad2): track 0.00 -> 14.6 mm
- net /12V_POST_RELAY: track 109.8 -> 99.2 mm
- net Net-(Q1-Pad1): track 9.79 -> 0.00 mm
- net Net-(R_EQ_V_DIV1-Pad1): track 0.00 -> 9.48 mm
- net Net-(R_EQ_V_DIV2-Pad2): track 4.70 -> 0.00 mm
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Other:
- board text added: "LedStripQ4’21 (v5) - ptab"
- board text removed: "LedStripQ1'21 (v4) - ptab"

Commit message: Link components to 3d images. Render back and front.
Other:
- net class 12V_15A removed
- net class Default removed
